Commit message: clean world file

File: urdf/my_robot.xacro (robot description, xacro)
@@ -124,5 +124,5 @@
     <inertial>
       <mass value="0.1"/>
-      <origin xyz="0.05 0.05 0.05"/>
+      <origin xyz="0.06 0.06 0.05"/>
       <inertia
           ixx="1e-6" ixy="0" ixz="0"
@@ -185,10 +185,10 @@
   </joint>
    <gazebo reference='left_wheel'>
-       <material>Gazebo/Green</material>
+       <material>Gazebo/White</material>
    </gazebo>
    <gazebo reference='right_wheel'>
-       <material>Gazebo/Green</material>
-   </gazebo>
-   <gazebo reference='chassis'>
+       <material>Gazebo/White</material>
+   </gazebo>
+   <gazebo reference="chassis">
        <material>Gazebo/Blue</material>
    </gazebo>
@@ -196,3 +196,6 @@
        <material>Gazebo/Red</material>
    </gazebo>
+   <gazebo reference="hokuyo">
+       <material>Gazebo/Green</material>
+   </gazebo>
 </robot>
