Commit message: added new rrRobot xacro file

File: urdf/rrRobot.xacro (robot description, xacro)
@@ -1,9 +1,9 @@
 <?xml version="1.0" ?>
-<robot name="my_robot">
+<robot name="my_robot" xmlns:xacro="http://www.ros.org/wiki/xacro">
 <!-- The root link robot_base has an inertia specified in the URDF,
  but KDL does not support a root link with an inertia.  As a workaround,
   adding an extra dummy link to URDF-->
   <link name="Dummy_link"></link>
-  <urdf:include filename="$(find my_robot)/urdf/my_robot.gazebo" />
+    <xacro:include filename="$(find my_robot)/urdf/my_robot.gazebo" />
   <joint name="Dummy_link_robot_base" type="fixed">
     <origin xyz="0 0 0" rpy="0 0 0" />
@@ -314,5 +314,5 @@
     </inertial>
     <collision name='camera_collision'>
-      <origin xyz="0 0 0" rpy="0 0  0"/>
+      <origin xyz="0 0 0" rpy="0 0 0"/>
       <geometry>
         <box size="0.05 0.05 0.05"/>
@@ -321,5 +321,5 @@
     </collision>
     <visual name='camera_visual'>
-      <origin xyz="0 0 0" rpy="0 0  0"/>
+      <origin xyz="0 0 0" rpy="0 0 0"/>
       <geometry>
         <box size="0.05 0.05 0.05"/>
@@ -329,8 +329,8 @@
   </link>
   <joint type="fixed" name="camera_joint">
-    <origin xyz="0.0 0.28 0.095" rpy="0 0 0"/>
+    <origin xyz="0.0 0.285 0.095" rpy="0 0 1.5707"/>
     <child link="camera"/>
     <parent link="robot_base"/>
-    <axis xyz="0 1 0" rpy="0 0 0"/>
+    <axis xyz="1 0 0" rpy="0 0 0"/>
   </joint>
    <gazebo reference='left_wheel'>

Commit message: corrected motion

File: urdf/rrRobot.xacro (robot description, xacro)
@@ -82,29 +82,35 @@
     <limit effort="0" lower="0" upper="0" velocity="0"/>
   </joint>
-  <link name="laser_scanner">
-    <inertial>
-      <mass value="1"/>
-      <origin rpy="0  0  0" xyz="0  0  0"/>
-      <inertia ixx="0.166667" ixy="0" ixz="0" iyy="0.166667" iyz="0" izz="0.166667"/>
-    </inertial>
-    <collision name="laser_scanner_collision">
-      <origin rpy="0    0.03  0" xyz="0  0  0"/>
-      <geometry>
-        <mesh filename="package://my_robot/meshes/hokuyo.dae" scale="1 1 1"/>
-      </geometry>
-    </collision>
-    <visual name="laser_scanner_visual">
-      <origin rpy="0    0.03  0" xyz="0  0  0"/>
-      <geometry>
-        <mesh filename="package://my_robot/meshes/hokuyo.dae" scale="1 1 1"/>
-      </geometry>
-    </visual>
-  </link>
-  <joint name="robot_base_laser_scanner" type="fixed">
-    <parent link="robot_base"/>
-    <child link="laser_scanner"/>
-    <origin rpy="-0.0001  -0.03725  0.01409" xyz="0  0 0.1500"/>
-    <axis xyz="0  0  0"/>
-    <limit effort="0" lower="0" upper="0" velocity="0"/>
+  <link name="hokuyo">
+    <pose>0 0 0 0 0 0</pose>
+    <inertial>
+      <mass value="1e-6"/>
+      <origin xyz="0.0 0 0" rpy=" 0 0 0"/>
+      <inertia
+          ixx="1e-6" ixy="0" ixz="0"
+          iyy="1e-6" iyz="0"
+          izz="1e-6"
+      />
+    </inertial>
+    <collision name='hokuyo_collision'>
+      <origin xyz="0.0 0 0" rpy=" 0 0 0"/>
+      <geometry>
+        <box size="0.1 0.1 0.1"/>
+      </geometry>
+      <mass value="1e-5"/>
+    </collision>
+    <visual name='hokuyo_visual'>
+      <origin xyz="0.0 0 0" rpy=" 0 0 0"/>
+      <geometry>
+        <mesh filename="package://my_robot/meshes/hokuyo.dae"/>
+      </geometry>
+      <mass value="1e-5"/>
+    </visual>
+  </link>
+  <joint type="fixed" name="hokuyo_joint">
+    <origin xyz="0.0 0 0.2" rpy="0 0 0"/>
+    <child link="hokuyo"/>
+    <parent link="robot_base"/>
+    <axis xyz="0 1 0" rpy="0 0 0"/>
   </joint>
   <link name="robot_left_support">
@@ -329,5 +335,5 @@
   </link>
   <joint type="fixed" name="camera_joint">
-    <origin xyz="0.0 0.285 0.095" rpy="0 0 1.5707"/>
+    <origin xyz="0.0 0.285 0.090" rpy="0 0 1.5707"/>
     <child link="camera"/>
     <parent link="robot_base"/>

Commit message: corrected CG

File: urdf/rrRobot.xacro (robot description, xacro)
@@ -13,5 +13,5 @@
   <link name="robot_base">
     <inertial>
-      <mass value="1"/>
+      <mass value="5"/>
       <origin rpy="0  0  0" xyz="0  0  0"/>
       <inertia ixx="0.145833" ixy="0" ixz="0" iyy="0.145833" iyz="0" izz="0.125"/>
@@ -32,5 +32,5 @@
   <link name="robot_middle_plate">
     <inertial>
-      <mass value="1"/>
+      <mass value="0.5"/>
       <origin rpy="0  0  0" xyz="0  0  0"/>
       <inertia ixx="0.145833" ixy="0" ixz="0" iyy="0.145833" iyz="0" izz="0.125"/>
@@ -58,5 +58,5 @@
   <link name="robot_top_plate">
     <inertial>
-      <mass value="1"/>
+      <mass value="0.3"/>
       <origin rpy="0  0  0" xyz="0  0  0"/>
       <inertia ixx="0.145833" ixy="0" ixz="0" iyy="0.145833" iyz="0" izz="0.125"/>
@@ -116,5 +116,5 @@
   <link name="robot_left_support">
     <inertial>
-      <mass value="1"/>
+      <mass value="0.1"/>
       <origin rpy="0  0  0" xyz="0  0  0"/>
       <inertia ixx="0.145833" ixy="0" ixz="0" iyy="0.145833" iyz="0" izz="0.125"/>
@@ -142,5 +142,5 @@
   <link name="robot_back_support">
     <inertial>
-      <mass value="1"/>
+      <mass value="0.1"/>
       <origin rpy="0  0  0" xyz="0  0  0"/>
       <inertia ixx="0.145833" ixy="0" ixz="0" iyy="0.145833" iyz="0" izz="0.125"/>
@@ -168,5 +168,5 @@
   <link name="robot_right_support">
     <inertial>
-      <mass value="1"/>
+      <mass value="0.1"/>
       <origin rpy="0  0  0" xyz="0  0  0"/>
       <inertia ixx="0.145833" ixy="0" ixz="0" iyy="0.145833" iyz="0" izz="0.125"/>
@@ -194,5 +194,5 @@
   <link name="front_caster">
     <inertial>
-      <mass value="1"/>
+      <mass value="0.1"/>
       <origin rpy="0  0  0" xyz="0  0  0"/>
       <inertia ixx="0.1" ixy="0" ixz="0" iyy="0.1" iyz="0" izz="0.1"/>
@@ -201,5 +201,5 @@
       <origin rpy="0  0  0" xyz="0  0  0"/>
       <geometry>
-        <sphere radius="0.055"/>
+        <sphere radius="0.0605"/>
       </geometry>
     </collision>
@@ -207,5 +207,5 @@
       <origin rpy="0  0  0" xyz="0  0  0"/>
       <geometry>
-        <sphere radius="0.055"/>
+        <sphere radius="0.0605"/>
       </geometry>
     </visual>
@@ -220,5 +220,5 @@
   <link name="back_caster">
     <inertial>
-      <mass value="1"/>
+      <mass value="0.1"/>
       <origin rpy="0  0  0" xyz="0  0  0"/>
       <inertia ixx="0.1" ixy="0" ixz="0" iyy="0.1" iyz="0" izz="0.1"/>
@@ -227,5 +227,5 @@
       <origin rpy="0  0  0" xyz="0  0  0"/>
       <geometry>
-        <sphere radius="0.055"/>
+        <sphere radius="0.0605"/>
       </geometry>
     </collision>
@@ -233,5 +233,5 @@
       <origin rpy="0  0  0" xyz="0  0  0"/>
       <geometry>
-        <sphere radius="0.055"/>
+        <sphere radius="0.0605"/>
       </geometry>
     </visual>
@@ -247,5 +247,5 @@
     <pose>0 0 0.1 0 0 0</pose>
     <inertial>
-      <mass value="5.0"/>
+      <mass value="1"/>
       <origin xyz="0.0 0 0" rpy="0 -1.5707  0"/>
       <inertia
@@ -279,5 +279,5 @@
     <pose>0 0 0.1 0 0 0</pose>
     <inertial>
-      <mass value="5.0"/>
+      <mass value="1.0"/>
       <origin xyz="0.0 0 0" rpy="0 1.5707  0"/>
       <inertia
@@ -335,5 +335,5 @@
   </link>
   <joint type="fixed" name="camera_joint">
-    <origin xyz="0.0 0.285 0.090" rpy="0 0 1.5707"/>
+    <origin xyz="0.0 0.285 0.060" rpy="0 0 1.5707"/>
     <child link="camera"/>
     <parent link="robot_base"/>
